Commit message: fix: XML typo in gripper_dark material

File: urdf/rebel_gripper_macro.xacro (robot description, xacro)
@@ -30,5 +30,5 @@
     </material>
     <material name="gripper_dark">
-        <color rgba="0.2 0.2 0.2 1.0" />I </material>
+        <color rgba="0.2 0.2 0.2 1.0" /></material>
     <material name="finger_color">
         <color rgba="0.79 0.82 0.93 1.0" />
